File: ESP32_Smart_Seedling_Waterer.kicad_pcb (KiCad board)
At the start: 2 copper layers, 84.3 x 51.3 mm, 23 parts, among them J1 Solenoid_12V, J2 AM2302 ~ DHT22, J3 Barrel_Jack_Switch, K1 SRD-05VDC-SL-C, Q1 PN2222A, Q2 PN2222A, SW1 SW_Push, SW3 SW_SPST, U1 LM7805_TO220, U2 ESP32-C3 SuperMini

Commit message: 9.5.2026 rtc added
Parts:
- added J4: DS3231 RTC, Connector_PinSocket_2.54mm:PinSocket_1x06_P2.54mm_Vertical, F.Cu at (144.7, 74.2)
- moved C3 10.1 mm to (179.2, 79.6)
- moved C4 10.1 mm to (174.4, 79.6)
- moved J2 10.1 mm to (179.5, 73.8)
- moved U2 8.31 mm to (157.5, 80.2)
- moved D1 5.18 mm to (169.8, 114.6)
- moved K1 5.18 mm to (143.7, 107.7)
- moved C1 5.18 mm to (126.1, 89.6)
- moved D3 5.18 mm to (115.9, 86.3)
- moved R4 5.18 mm to (117.8, 111.3)
- moved R6 5.18 mm to (128.0, 115.3)
- moved SW1 5.18 mm to (106.6, 112.1)
- moved D2 5.18 mm to (107.9, 101.0)
- moved R5 5.18 mm to (128.0, 105.2)
- moved U1 5.18 mm to (129.8, 91.4)
- moved C2 5.18 mm to (138.6, 89.8)
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Connections:
- net Net-(J2-Pin_2) renamed +3V3
- U2 pad 2: unconnected-(U2-GPIO6-Pad2) -> Net-(J4-Pin_3)
- U2 pad 3: unconnected-(U2-GPIO7-Pad3) -> Net-(J4-Pin_4)
Routing:
- net +3V3: track 11.5 -> 82.9 mm
- net +5V: track 256.1 -> 273.4 mm
- net GND: track 311.8 -> 326.9 mm
- net Net-(J4-Pin_4): track 0.00 -> 6.47 mm
- net Net-(J4-Pin_3): track 0.00 -> 6.47 mm
- net SW_WATER: track 92.2 -> 95.6 mm
- net +12V: track 92.8 -> 95.4 mm
- net Net-(J2-Pin_1): track 15.1 -> 17.4 mm
Other:
- board size 84.3 x 51.3 mm -> 83.8 x 51.8 mm
